Commit message: osr_gazebo: simple collision shapes for Gazebo Harmonic (stage 5 of port)
The URDF used the detailed CAD meshes as collision geometry (~1M triangles,
body.stl alone 218k), which held the Harmonic sim to ~58% real time. With
sim:=harmonic the drive wheels now collide as cylinders sized from wheel.stl
(r 82 mm, w 101 mm), the body as a box matching its outer dimensions, and the
remaining links have no collision shape. Visuals still use the meshes.
Gazebo Classic output is unchanged (verified with canonicalized xacro output).

Co-Authored-By: Claude Opus 5.5 <noreply@anthropic.com>
Claude-Session: https://claude.ai/code/session_018TQRf6V6R8o2WMQezLAfNd

File: ROS/osr_gazebo/urdf/osr.urdf.xacro (robot description, xacro)
@@ -21,12 +21,34 @@
     <xacro:include filename="$(find osr_gazebo)/urdf/gazebo.urdf.xacro"/>
     <xacro:include filename="$(find osr_gazebo)/urdf/insert_transmission.urdf.xacro"/>
+    <!-- Collision shapes. Gazebo Classic uses the detailed CAD meshes for collisions
+         (unchanged from upstream). In Harmonic, colliding ~1 million mesh triangles
+         with the ground every physics step made the sim run at about half real time,
+         so there the drive wheels collide as simple cylinders, the body as a box, and
+         the other links (rocker-bogie, steering brackets) have no collision shape: on
+         flat ground only the wheels touch anything. Visuals still use the meshes.
+         Cylinder sized from wheel.stl: radius 82 mm, width 101 mm, centered 7.5 mm
+         off the link origin along the axle. -->
+    <xacro:property name="wheel_collision_radius" value="0.082"/>
+    <xacro:property name="wheel_collision_width" value="0.101"/>
+    <xacro:property name="wheel_collision_offset" value="-0.0075"/>
     <link name="base_footprint"/>
     <link name="base_link">
-        <collision>
-            <origin rpy="0 0 0" xyz="0 0 0.0"/>
-            <geometry>
-                <mesh filename="file://$(find osr_gazebo)/meshes/body.stl"/>
-            </geometry>
-        </collision>
+        <xacro:if value="${sim == 'classic'}">
+            <collision>
+                        <origin rpy="0 0 0" xyz="0 0 0.0"/>
+                        <geometry>
+                            <mesh filename="file://$(find osr_gazebo)/meshes/body.stl"/>
+                        </geometry>
+                    </collision>
+        </xacro:if>
+        <xacro:if value="${sim == 'harmonic'}">
+            <!-- Box matching the body's outer dimensions -->
+            <collision>
+                <origin rpy="0 0 0" xyz="0 0 0.0115"/>
+                <geometry>
+                    <box size="0.356 0.254 0.141"/>
+                </geometry>
+            </collision>
+        </xacro:if>
         <visual>
             <origin rpy="0 0 0" xyz="0 0 0.0"/>
@@ -49,10 +71,12 @@
     </joint>
     <link name="box_rotate">
-        <collision>
-            <origin rpy="0 0 -3.14" xyz="0 0 0.0"/>
-            <geometry>
-                <mesh filename="file://$(find osr_gazebo)/meshes/box_link.stl"/>
-            </geometry>
-        </collision>
+        <xacro:if value="${sim == 'classic'}">
+            <collision>
+                        <origin rpy="0 0 -3.14" xyz="0 0 0.0"/>
+                        <geometry>
+                            <mesh filename="file://$(find osr_gazebo)/meshes/box_link.stl"/>
+                        </geometry>
+                    </collision>
+        </xacro:if>
         <visual>
             <origin rpy="0 0 -3.14" xyz="0 0 0"/>
@@ -76,10 +100,12 @@
     <xacro:macro name="arm_rotate" params="prefix dir">
         <link name="arm_rotate_${prefix}">
-            <collision>
-                <origin rpy="0 0.2 0" xyz="0 0 0"/>
-                <geometry>
-                    <mesh filename="file://$(find osr_gazebo)/meshes/arm.stl"/>
-                </geometry>
-            </collision>
+            <xacro:if value="${sim == 'classic'}">
+                <collision>
+                                <origin rpy="0 0.2 0" xyz="0 0 0"/>
+                                <geometry>
+                                    <mesh filename="file://$(find osr_gazebo)/meshes/arm.stl"/>
+                                </geometry>
+                            </collision>
+            </xacro:if>
             <visual>
                 <origin rpy="0 0.2 0" xyz="0 0 0"/>
@@ -106,10 +132,12 @@
     <xacro:macro name="turn_bukles" params="prefix dir origin">
         <link name="turn_bukles_link_${prefix}">
-            <collision>
-                <origin rpy="0 0 ${origin}" xyz="0 0 0.0"/>
-                <geometry>
-                    <mesh filename="file://$(find osr_gazebo)/meshes/turn_${prefix}.stl"/>
-                </geometry>
-            </collision>
+            <xacro:if value="${sim == 'classic'}">
+                <collision>
+                                <origin rpy="0 0 ${origin}" xyz="0 0 0.0"/>
+                                <geometry>
+                                    <mesh filename="file://$(find osr_gazebo)/meshes/turn_${prefix}.stl"/>
+                                </geometry>
+                            </collision>
+            </xacro:if>
             <visual>
                 <origin rpy="0 0 ${origin}" xyz="0 0 0.0"/>
@@ -136,10 +164,12 @@
     <xacro:macro name="body_axis_link" params="prefix dir">
         <link name="body_axis_link_${prefix}">
-            <collision>
-                <origin rpy="0 0 1.57" xyz="0 0 0.0"/>
-                <geometry>
-                    <mesh filename="file://$(find osr_gazebo)/meshes/body_axis.stl"/>
-                </geometry>
-            </collision>
+            <xacro:if value="${sim == 'classic'}">
+                <collision>
+                                <origin rpy="0 0 1.57" xyz="0 0 0.0"/>
+                                <geometry>
+                                    <mesh filename="file://$(find osr_gazebo)/meshes/body_axis.stl"/>
+                                </geometry>
+                            </collision>
+            </xacro:if>
             <visual>
                 <origin rpy="0 0 1.57" xyz="0 0 0.0"/>
@@ -166,10 +196,12 @@
     <xacro:macro name="rocker_bogie_link" params="prefix dir">
         <link name="rocker_bogie_link_${prefix}_1">
-            <collision>
-                <origin rpy="0 0 0" xyz="0 0 0.0"/>
-                <geometry>
-                    <mesh filename="file://$(find osr_gazebo)/meshes/rockerbogie_middle_1.stl"/>
-                </geometry>
-            </collision>
+            <xacro:if value="${sim == 'classic'}">
+                <collision>
+                                <origin rpy="0 0 0" xyz="0 0 0.0"/>
+                                <geometry>
+                                    <mesh filename="file://$(find osr_gazebo)/meshes/rockerbogie_middle_1.stl"/>
+                                </geometry>
+                            </collision>
+            </xacro:if>
             <visual>
                 <origin rpy="0 0 0" xyz="0 0 0.0"/>
@@ -193,10 +225,12 @@
         </joint>
         <link name="rocker_bogie_link_${prefix}_2">
-            <collision>
-                <origin rpy="0 0 0" xyz="0 0 0.0"/>
-                <geometry>
-                    <mesh filename="file://$(find osr_gazebo)/meshes/rockerbogie_front_1.stl"/>
-                </geometry>
-            </collision>
+            <xacro:if value="${sim == 'classic'}">
+                <collision>
+                                <origin rpy="0 0 0" xyz="0 0 0.0"/>
+                                <geometry>
+                                    <mesh filename="file://$(find osr_gazebo)/meshes/rockerbogie_front_1.stl"/>
+                                </geometry>
+                            </collision>
+            </xacro:if>
             <visual>
                 <origin rpy="0 0 0" xyz="0 0 0.0"/>
@@ -224,10 +258,12 @@
     <xacro:macro name="wheel_link" params="prefix dir origin">
         <link name="front_wheel_link_${prefix}">
-            <collision>
-                <origin rpy="0 0 ${dir*-1.57}" xyz="0 0 0.0"/>
-                <geometry>
-                    <mesh filename="file://$(find osr_gazebo)/meshes/wheel_link_left_2.stl"/>
-                </geometry>
-            </collision>
+            <xacro:if value="${sim == 'classic'}">
+                <collision>
+                                <origin rpy="0 0 ${dir*-1.57}" xyz="0 0 0.0"/>
+                                <geometry>
+                                    <mesh filename="file://$(find osr_gazebo)/meshes/wheel_link_left_2.stl"/>
+                                </geometry>
+                            </collision>
+            </xacro:if>
             <visual>
                 <origin rpy="0 0 ${dir*-1.57}" xyz="0 0 0.0"/>
@@ -252,10 +288,12 @@
         </joint>
         <link name="middle_wheel_link_${prefix}">
-            <collision>
-                <origin rpy="${origin} 0 ${-dir*1.57}" xyz="0 0 0.0"/>
-                <geometry>
-                    <mesh filename="file://$(find osr_gazebo)/meshes/wheel_middle_left.stl"/>
-                </geometry>
-            </collision>
+            <xacro:if value="${sim == 'classic'}">
+                <collision>
+                                <origin rpy="${origin} 0 ${-dir*1.57}" xyz="0 0 0.0"/>
+                                <geometry>
+                                    <mesh filename="file://$(find osr_gazebo)/meshes/wheel_middle_left.stl"/>
+                                </geometry>
+                            </collision>
+            </xacro:if>
             <visual>
                 <origin rpy="${origin} 0 ${-dir*1.57}" xyz="0 0 0.0"/>
@@ -278,10 +316,12 @@
         </joint>
         <link name="rear_wheel_link_${prefix}">
-            <collision>
-                <origin rpy="0 0 ${-dir*1.57}" xyz="0 0 0.0"/>
-                <geometry>
-                    <mesh filename="file://$(find osr_gazebo)/meshes/wheel_link_left_2.stl"/>
-                </geometry>
-            </collision>
+            <xacro:if value="${sim == 'classic'}">
+                <collision>
+                                <origin rpy="0 0 ${-dir*1.57}" xyz="0 0 0.0"/>
+                                <geometry>
+                                    <mesh filename="file://$(find osr_gazebo)/meshes/wheel_link_left_2.stl"/>
+                                </geometry>
+                            </collision>
+            </xacro:if>
             <visual>
                 <origin rpy="0 0 ${-dir*1.57}" xyz="0 0 0.0"/>
@@ -322,10 +362,21 @@
         <xacro:wheel_friction link="rear_wheel_link_${prefix}"/>
         <link name="front_wheel_link_${prefix}">
-            <collision>
-                <origin rpy="-1.57 0 ${origin}" xyz="0 0 0.0"/>
-                <geometry>
-                    <mesh filename="file://$(find osr_gazebo)/meshes/wheel.stl"/>
-                </geometry>
-            </collision>
+            <xacro:if value="${sim == 'classic'}">
+                <collision>
+                                <origin rpy="-1.57 0 ${origin}" xyz="0 0 0.0"/>
+                                <geometry>
+                                    <mesh filename="file://$(find osr_gazebo)/meshes/wheel.stl"/>
+                                </geometry>
+                            </collision>
+            </xacro:if>
+            <xacro:if value="${sim == 'harmonic'}">
+                <!-- Simple cylinder instead of the detailed tire mesh (see note at top) -->
+                <collision>
+                    <origin rpy="1.5708 0 0" xyz="0 ${wheel_collision_offset * cos(origin)} 0"/>
+                    <geometry>
+                        <cylinder radius="${wheel_collision_radius}" length="${wheel_collision_width}"/>
+                    </geometry>
+                </collision>
+            </xacro:if>
             <visual>
                 <origin rpy="-1.57 0 ${origin}" xyz="0 0 0.0"/>
@@ -349,10 +400,21 @@
         </joint>
         <link name="middle_wheel_link_${prefix}">
-            <collision>
-                <origin rpy="-1.57 0 ${origin}" xyz="0 0 0.0"/>
-                <geometry>
-                    <mesh filename="file://$(find osr_gazebo)/meshes/wheel.stl"/>
-                </geometry>
-            </collision>
+            <xacro:if value="${sim == 'classic'}">
+                <collision>
+                                <origin rpy="-1.57 0 ${origin}" xyz="0 0 0.0"/>
+                                <geometry>
+                                    <mesh filename="file://$(find osr_gazebo)/meshes/wheel.stl"/>
+                                </geometry>
+                            </collision>
+            </xacro:if>
+            <xacro:if value="${sim == 'harmonic'}">
+                <!-- Simple cylinder instead of the detailed tire mesh (see note at top) -->
+                <collision>
+                    <origin rpy="1.5708 0 0" xyz="0 ${wheel_collision_offset * cos(origin)} 0"/>
+                    <geometry>
+                        <cylinder radius="${wheel_collision_radius}" length="${wheel_collision_width}"/>
+                    </geometry>
+                </collision>
+            </xacro:if>
             <visual>
                 <origin rpy="-1.57 0 ${origin}" xyz="0 0 0.0"/>
@@ -376,10 +438,21 @@
         </joint>
         <link name="rear_wheel_link_${prefix}">
-            <collision>
-                <origin rpy="-1.57 0 ${origin}" xyz="0 0 0.0"/>
-                <geometry>
-                    <mesh filename="file://$(find osr_gazebo)/meshes/wheel.stl"/>
-                </geometry>
-            </collision>
+            <xacro:if value="${sim == 'classic'}">
+                <collision>
+                                <origin rpy="-1.57 0 ${origin}" xyz="0 0 0.0"/>
+                                <geometry>
+                                    <mesh filename="file://$(find osr_gazebo)/meshes/wheel.stl"/>
+                                </geometry>
+                            </collision>
+            </xacro:if>
+            <xacro:if value="${sim == 'harmonic'}">
+                <!-- Simple cylinder instead of the detailed tire mesh (see note at top) -->
+                <collision>
+                    <origin rpy="1.5708 0 0" xyz="0 ${wheel_collision_offset * cos(origin)} 0"/>
+                    <geometry>
+                        <cylinder radius="${wheel_collision_radius}" length="${wheel_collision_width}"/>
+                    </geometry>
+                </collision>
+            </xacro:if>
             <visual>
                 <origin rpy="-1.57 0 ${origin}" xyz="0 0 0.0"/>
