Commit message: osr_gazebo: drive wheels and steering in Gazebo Harmonic (stage 3 of port)
- gazebo.urdf.xacro: one shared ros2_control joint description; the hardware
  plugin is gazebo_ros2_control/GazeboSystem for sim:=classic and
  gz_ros2_control/GazeboSimSystem for sim:=harmonic, with the matching
  simulator plugin for each. Classic IMU plugin stays Classic-only.
  Classic xacro output is unchanged.
- config/controllers_harmonic.yaml: same controllers as Classic, but the
  steering controller claims only the position interface (claiming position
  and velocity together makes gz_ros2_control drive the joint from both)
- harmonic_world.launch.py: spawn joint_state_broadcaster, wheel_controller
  and servo_controller
- package.xml: exec_depend on gz_ros2_control and controller_manager

Co-Authored-By: Claude Opus 5.5 <noreply@anthropic.com>
Claude-Session: https://claude.ai/code/session_018TQRf6V6R8o2WMQezLAfNd

File: ROS/osr_gazebo/urdf/gazebo.urdf.xacro (robot description, xacro)
@@ -1,11 +1,16 @@
 <?xml version="1.0"?>
 <robot xmlns:xacro="http://wiki.ros.org/xacro">
-  <!-- Gazebo Classic plugins (gazebo_ros2_control, Classic IMU plugin).
-       Harmonic equivalents are added separately; until then a Harmonic run
-       loads only the physical model. -->
-  <xacro:if value="${'$(arg sim)' == 'classic'}">
+  <!-- ros2_control describes what each joint can be commanded with. The joint list is
+       the same for both simulators; only the hardware plugin that plays "the robot"
+       differs: gazebo_ros2_control for Gazebo Classic, gz_ros2_control for Harmonic. -->
+  <xacro:property name="sim" value="$(arg sim)"/>
   <ros2_control name="GazeboSystem" type="system">
     <hardware>
-      <plugin>gazebo_ros2_control/GazeboSystem</plugin>
+      <xacro:if value="${sim == 'classic'}">
+        <plugin>gazebo_ros2_control/GazeboSystem</plugin>
+      </xacro:if>
+      <xacro:if value="${sim == 'harmonic'}">
+        <plugin>gz_ros2_control/GazeboSimSystem</plugin>
+      </xacro:if>
     </hardware>
     <joint name="middle_wheel_joint_left">
@@ -115,9 +120,20 @@
     </joint>
   </ros2_control>
-  <gazebo>
-    <plugin filename="libgazebo_ros2_control.so" name="gazebo_ros2_control">
-      <parameters>$(find osr_gazebo)/config/controller_velocity.yaml</parameters>
-    </plugin>
-  </gazebo>
+  <xacro:if value="${sim == 'classic'}">
+    <gazebo>
+      <plugin filename="libgazebo_ros2_control.so" name="gazebo_ros2_control">
+        <parameters>$(find osr_gazebo)/config/controller_velocity.yaml</parameters>
+      </plugin>
+    </gazebo>
+  </xacro:if>
+  <xacro:if value="${sim == 'harmonic'}">
+    <gazebo>
+      <plugin filename="gz_ros2_control-system" name="gz_ros2_control::GazeboSimROS2ControlPlugin">
+        <parameters>$(find osr_gazebo)/config/controllers_harmonic.yaml</parameters>
+      </plugin>
+    </gazebo>
+  </xacro:if>
+  <!-- Gazebo Classic IMU plugin; a Harmonic IMU sensor is a later step -->
+  <xacro:if value="${sim == 'classic'}">
     <gazebo reference="imu_link">
         <gravity>true</gravity>

Commit message: osr_gazebo: report bogie pivot angles so the full rover shows in RViz
In Harmonic, joint_state_broadcaster only publishes joints listed in the
ros2_control block. The passive bogie pivots (rocker_bogie_joint_L_2/R_2)
weren't, so robot_state_publisher had no transform for the bogies and
everything mounted on them: RViz showed the front and middle wheels missing
("No transform from front_wheel_link_R"). Add them as state-only joints
(harmonic only; Classic output unchanged).

Co-Authored-By: Claude Opus 5.5 <noreply@anthropic.com>
Claude-Session: https://claude.ai/code/session_018TQRf6V6R8o2WMQezLAfNd

File: ROS/osr_gazebo/urdf/gazebo.urdf.xacro (robot description, xacro)
@@ -119,4 +119,17 @@
       <state_interface name="effort"/>
     </joint>
+    <!-- Passive bogie pivots: not driven, but their angles must be reported so
+         robot_state_publisher can place the bogie and everything mounted on it
+         (front and middle wheels) in TF. State interfaces only, no command. -->
+    <xacro:if value="${sim == 'harmonic'}">
+      <joint name="rocker_bogie_joint_L_2">
+        <state_interface name="position"/>
+        <state_interface name="velocity"/>
+      </joint>
+      <joint name="rocker_bogie_joint_R_2">
+        <state_interface name="position"/>
+        <state_interface name="velocity"/>
+      </joint>
+    </xacro:if>
   </ros2_control>
   <xacro:if value="${sim == 'classic'}">
